File: Hardware/ADJD-S311_Breakout.brd (EAGLE design)
At the start: 23.2 x 12.7 mm, 21 parts, among them Q2 MMBT2222, U1 ADJD-S311-CR999V2, U2 2.8V, U3 2.8V

Commit message: Fixed footprint to testing
Parts:
- added U$1: REVISION, SparkFun-Aesthetics:REVISION
- U1: value ADJD-S311-CR999V2 -> ADJD-S311-CR999; device Testing:CSP-9-V2 -> SparkFun-Sensors:CSP-9
Routing:
- net GND: track 31.0 -> 28.8 mm
Other:
- board text added: "N. Seidle"
- board text added: "T. Klopfenstein"
- board text removed: "N. Seidle, Revision by: T. Klopfenstein"
Changed lines of the file:
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@@
 <layer number="106" name="bPlate" color="7" fill="1" visible="no" active="yes"/>
 <layer number="107" name="Crop" color="7" fill="1" visible="no" active="yes"/>
+<layer number="108" name="tplace-old" color="10" fill="1" visible="no" active="yes"/>
+<layer number="109" name="ref-old" color="11" fill="1" visible="no" active="yes"/>
 <layer number="116" name="Patch_BOT" color="9" fill="4" visible="no" active="yes"/>
 <layer number="121" name="_tsilk" color="7" fill="1" visible="no" active="yes"/>
@@
 <text x="20.193" y="5.715" size="1.27" layer="22" font="vector" ratio="15" rot="MR0">SLP</text>
 <text x="20.193" y="3.175" size="1.27" layer="22" font="vector" ratio="15" rot="MR0">CLK</text>
-<text x="24.13" y="-11.43" size="1.778" layer="25" font="vector" ratio="15">N. Seidle, Revision by:  T. Klopfenstein</text>
+<text x="24.13" y="-11.43" size="1.778" layer="25" font="vector" ratio="15">N. Seidle</text>
 <text x="22.2885" y="0.635" size="1.27" layer="22" font="vector" ratio="15" rot="MR0">ADJD-S311</text>
 <text x="22.225" y="11.43" size="0.8128" layer="16" font="vector" ratio="25" rot="MR0">v12</text>
+<text x="24.13" y="-13.97" size="1.778" layer="25" font="vector" ratio="15">T. Klopfenstein</text>
 </plain>
 <attributes>
@@
 <element name="JP2" library="SparkFun" package="SFE-LOGO-FLAME" value="LOGO-SFESK" x="17.78" y="1.27"/>
 <element name="JP4" library="SparkFun" package="1X05" value="" x="1.27" y="11.43" rot="R270"/>
-<element name="U1" library="Testing" package="CSP-9-V2" value="ADJD-S311-CR999V2" x="13.97" y="6.35" rot="R180"/>
+<element name="U1" library="SparkFun-Sensors" package="CSP-9" value="ADJD-S311-CR999" x="13.97" y="6.35" rot="R180"/>
 <element name="U$4" library="SparkFun" package="OSHW-LOGO-S" value="OSHW-LOGOS" x="15.24" y="2.667"/>
 <element name="JP1" library="SparkFun" package="SFE-LOGO-FLAME" value="LOGO-SFESK" x="11.811" y="4.699" rot="MR0"/>
 <element name="FRAME1" library="SparkFun-Aesthetics" package="CREATIVE_COMMONS" value="FRAME-LETTER" x="-7.092121875" y="-11.43"/>
+<element name="U$1" library="SparkFun-Aesthetics" package="REVISION" value="REVISION" x="4.318" y="-13.97"/>
 </elements>
 <signals>
@@
 <contactref element="U1" pad="C1"/>
 <contactref element="Q2" pad="2"/>
-<wire x1="14.53" y1="6.91" x2="14.53" y2="7.926" width="0.254" layer="1"/>
-<wire x1="14.53" y1="7.926" x2="14.732" y2="8.128" width="0.254" layer="1"/>
-<wire x1="14.53" y1="6.91" x2="15.419" y2="6.91" width="0.254" layer="1"/>
 <wire x1="15.419" y1="6.91" x2="15.494" y2="6.985" width="0.254" layer="1"/>
 <wire x1="15.494" y1="6.985" x2="15.494" y2="7.366" width="0.254" layer="1"/>
@@
 <vertex x="23.1775" y="0"/>
 </polygon>
-<wire x1="13.41" y1="6.91" x2="11.43" y2="8.89" width="0.2032" layer="1"/>
+<wire x1="13.41" y1="6.9354" x2="11.43" y2="8.89" width="0.2032" layer="1"/>
 <wire x1="8.3575" y1="3.175" x2="7.493" y2="3.175" width="0.254" layer="1"/>
 <wire x1="7.493" y1="3.175" x2="7.366" y2="3.302" width="0.254" layer="1"/>
@@
 <wire x1="11.3665" y1="3.175" x2="10.0575" y2="3.175" width="0.254" layer="1"/>
 <wire x1="10.0575" y1="3.175" x2="10.0575" y2="1.5875" width="0.254" layer="1"/>
-<wire x1="13.41" y1="5.79" x2="13.41" y2="4.647" width="0.2032" layer="1"/>
+<wire x1="13.41" y1="5.8408" x2="13.41" y2="4.647" width="0.2032" layer="1"/>
 <wire x1="13.41" y1="4.647" x2="11.938" y2="3.175" width="0.2032" layer="1"/>
 <wire x1="11.938" y1="3.175" x2="11.3665" y2="3.175" width="0.2032" layer="1"/>
@@
 <contactref element="R1" pad="1"/>
 <contactref element="U1" pad="C2"/>
-<wire x1="13.97" y1="6.91" x2="13.97" y2="7.62" width="0.254" layer="1"/>
 <wire x1="13.97" y1="7.62" x2="10.4775" y2="11.1125" width="0.254" layer="1"/>
 <wire x1="10.4775" y1="11.1125" x2="10.0575" y2="11.1125" width="0.254" layer="1"/>
+<wire x1="13.9446" y1="6.9354" x2="13.9446" y2="7.5946" width="0.254" layer="1"/>
+<wire x1="13.9446" y1="7.5946" x2="13.97" y2="7.62" width="0.2032" layer="1"/>
 </signal>
 <signal name="SDA">
@@
 <wire x1="15.24" y1="3.175" x2="15.24" y2="3.2004" width="0.127" layer="1"/>
 <wire x1="15.24" y1="3.2004" x2="14.2494" y2="4.191" width="0.127" layer="1"/>
-<wire x1="13.97" y1="6.35" x2="13.9954" y2="6.35" width="0.127" layer="1"/>
+<wire x1="13.9446" y1="6.3754" x2="13.9954" y2="6.35" width="0.127" layer="1"/>
 <wire x1="13.9954" y1="6.35" x2="14.2494" y2="6.096" width="0.127" layer="1"/>
 <wire x1="14.2494" y1="6.096" x2="14.2494" y2="4.191" width="0.127" layer="1"/>
@@
 <contactref element="U1" pad="A2"/>
 <wire x1="1.27" y1="3.81" x2="3.81" y2="3.81" width="0.2032" layer="16"/>
-<wire x1="13.97" y1="5.79" x2="13.97" y2="5.842" width="0.127" layer="1"/>
+<wire x1="13.97" y1="5.8408" x2="13.97" y2="5.842" width="0.127" layer="1"/>
 <wire x1="9.652" y1="4.572" x2="9.652" y2="5.715" width="0.2032" layer="16"/>
 <wire x1="10.287" y1="3.937" x2="9.652" y2="4.572" width="0.2032" layer="16"/>
@@
 <via x="13.6525" y="3.175" extent="1-16" drill="0.381"/>
 <via x="11.43" y="6.03123125" extent="1-16" drill="0.381"/>
-<wire x1="13.97" y1="5.79" x2="13.97" y2="3.4925" width="0.1524" layer="1"/>
+<wire x1="13.97" y1="5.8408" x2="13.97" y2="3.4925" width="0.1524" layer="1"/>
 <wire x1="13.97" y1="3.4925" x2="13.6525" y2="3.175" width="0.254" layer="1"/>
 <wire x1="13.6525" y1="3.175" x2="13.335" y2="3.175" width="0.254" layer="16"/>
@@
 <contactref element="JP3" pad="3"/>
 <contactref element="U1" pad="B1"/>
-<wire x1="14.53" y1="6.35" x2="19.939" y2="6.35" width="0.2032" layer="1"/>
-<wire x1="19.939" y1="6.35" x2="20.193" y2="6.096" width="0.2032" layer="1"/>
+<wire x1="19.9136" y1="6.3754" x2="20.193" y2="6.096" width="0.2032" layer="1"/>
 <wire x1="20.193" y1="6.096" x2="20.193" y2="5.207" width="0.2032" layer="1"/>
 <wire x1="20.193" y1="5.207" x2="21.59" y2="3.81" width="0.2032" layer="1"/>
+<wire x1="14.4792" y1="6.3754" x2="19.9136" y2="6.3754" width="0.2032" layer="1"/>
 </signal>
 <signal name="SLEEP">
@@
 <wire x1="19.05" y1="7.2" x2="20.74" y2="7.2" width="0.254" layer="1"/>
 <wire x1="20.74" y1="7.2" x2="21.59" y2="6.35" width="0.254" layer="1"/>
-<wire x1="13.41" y1="6.35" x2="12.827" y2="6.35" width="0.2032" layer="1"/>
-<wire x1="12.827" y1="6.35" x2="11.43" y2="7.747" width="0.2032" layer="1"/>
+<wire x1="13.41" y1="6.3754" x2="12.8016" y2="6.3754" width="0.2032" layer="1"/>
+<wire x1="12.8016" y1="6.3754" x2="11.43" y2="7.747" width="0.2032" layer="1"/>
 </signal>
 <signal name="2.8V">
@@
 <wire x1="6.35" y1="8.89" x2="6.35" y2="8.636" width="0.2032" layer="16"/>
 <wire x1="6.35" y1="8.636" x2="8.001" y2="6.985" width="0.2032" layer="16"/>
-<wire x1="14.53" y1="5.79" x2="15.248821875" y2="5.79" width="0.2032" layer="1"/>
-<wire x1="15.248821875" y1="5.79" x2="15.61973125" y2="5.419090625" width="0.2032" layer="1"/>
+<wire x1="15.198021875" y1="5.8408" x2="15.61973125" y2="5.419090625" width="0.2032" layer="1"/>
 <wire x1="15.61973125" y1="5.419090625" x2="15.61973125" y2="4.509771875" width="0.2032" layer="1"/>
 <wire x1="15.61973125" y1="4.509771875" x2="15.55623125" y2="4.446271875" width="0.2032" layer="1"/>
@@
 <wire x1="8.3575" y1="11.1125" x2="7.6526" y2="11.1125" width="0.2032" layer="1"/>
 <wire x1="7.6526" y1="11.1125" x2="6.3801" y2="9.84" width="0.2032" layer="1"/>
+<wire x1="14.4792" y1="5.8408" x2="15.198021875" y2="5.8408" width="0.2032" layer="1"/>
 </signal>
 <signal name="N$3">
